Commit message: feat(sim): integrate V6 patrol robot and perception pipeline

File: ros_ws/src/metro_description/urdf/subway_v2.urdf (robot description, URDF)
Before this commit: robot subway_v2, 31 links, 30 joints
Links:
- removed link w1_hub
- removed link w2_hub
- removed link w3_hub
- removed link w4_hub
- link base_link: mass 14.4385473688281 -> 15.4748516352473; geometry collision box size=0.475999981165 0.276014514267 0.464500010014; visual mesh filename=package://metro_description/meshes/base_link.STL
- link leida: mass 0.224138920024067 -> 0.224138920084812; geometry collision box size=0.100000001490 0.061999998987 0.046399998944
- link pitch: geometry collision box size=0.193599997088 0.122999997810 0.234749644995; visual mesh filename=package://metro_description/meshes/pitch.STL
- link pitch_camera: mass 0.001 -> None; geometry 
- link w1: mass 0.432839204473948 -> 0.5; geometry collision cylinder length=0.013 radius=0.0775; collision cylinder length=0.019 radius=0.060
- link w2: mass 0.432839204200384 -> 0.5; geometry collision cylinder length=0.013 radius=0.0775; collision cylinder length=0.019 radius=0.060
- link w3: mass 0.432839204470938 -> 0.5; geometry collision cylinder length=0.013 radius=0.0775; collision cylinder length=0.019 radius=0.060
- link w4: mass 0.432839204102094 -> 0.5; geometry collision cylinder length=0.013 radius=0.0775; collision cylinder length=0.019 radius=0.060
- link xj1: geometry collision box size=0.037850178778 0.057438004762 0.120107173920; visual mesh filename=package://metro_description/meshes/xj1.STL
- link xj2: geometry collision box size=0.037850178778 0.057438004762 0.120107173920; visual mesh filename=package://metro_description/meshes/xj2.STL
- link xj3: mass 0.0702201485513357 -> 0.0702201485513358; geometry collision box size=0.037850178778 0.037925016135 0.115999998525; visual mesh filename=package://metro_description/meshes/xj3.STL
- link xj4: geometry collision box size=0.037850178778 0.037925016135 0.115999998525; visual mesh filename=package://metro_description/meshes/xj4.STL
- link yuntai: geometry collision box size=0.140000000596 0.218761026859 0.191999999806; visual mesh filename=package://metro_description/meshes/yuntai.STL
Joints:
- removed joint ld
- removed joint ph
- removed joint w1_hub_joint
- removed joint w2_hub_joint
- removed joint w3_hub_joint
- removed joint w4_hub_joint
- removed joint yaw
- added joint leida_joint: type fixed, parent base_link, child leida, origin xyz=0.00342893995182154 -0.0120000000000005 0.139095970953207 rpy=0 0 0, axis 0 0 0
- added joint pitch_joint: type fixed, parent yuntai, child pitch, origin xyz=0 0.01 0 rpy=3.14050535389669 -1.5707963267949 0
- added joint yaw_joint: type fixed, parent base_link, child yuntai, origin xyz=-0.0738710600481814 -0.166 -0.0109040290468001 rpy=3.14159265358979 1.5707963267949 0
- joint base_footprint_to_base_link: origin xyz=0 0 0 rpy=-1.5707963267949 0 -1.5707963267949 -> xyz=0.010904028627 0.003428939952 0.214499211212 rpy=-1.570796326795 0 -1.570796326795
- joint lidar_joint: origin xyz=-0.0055 0 0.0078 rpy=1.5707963267949 -1.5707963267949 0 -> xyz=0 0 0.041 rpy=1.5707963267949 -1.5707963267949 0
- joint pitch_camera_optical_joint: origin xyz=0 0 0 rpy=-1.5707963267949 0 -1.5707963267949 -> xyz=0 0 0 rpy=-1.570796326795 0 -1.570796326795
- joint pitch_camera_sensor_joint: origin xyz=-0.077300002798 0.003299999982 0.087818765 rpy=-1.5707963267949 -1.5707963267949 0 -> xyz=-0.077300002798 0.003299999982 0.087818765 rpy=1.5707963267949 -1.5707963267949 0
- joint w1_joint: origin xyz=0.152328939951822 0.103 0.134095970953207 rpy=1.57079632679489 -0.16843576907617 1.5707963267949 -> xyz=0.254228939952 0.136999998856323 0.134095974152992 rpy=1.57079632679489 -0.16843576907617 1.5707963267949
- joint w2_joint: axis 0 0 -1 -> 0 0 1; origin xyz=-0.145471060048178 0.103 0.134095970953207 rpy=1.57079632679489 0.16843576907617 -1.5707963267949 -> xyz=-0.247371060048 0.136999998934387 0.134095970636500 rpy=1.57079632679489 0.16843576907617 -1.5707963267949
- joint w3_joint: axis 0 0 -1 -> 0 0 1; origin xyz=-0.145471060048178 0.102999999999999 -0.155904029046793 rpy=1.57079632679489 1.06806361303278 -1.5707963267949 -> xyz=-0.247371060048 0.136999999067289 -0.155904029760880 rpy=1.57079632679489 1.06806361303278 -1.5707963267949
- joint w4_joint: origin xyz=0.152328939951822 0.102999999999999 -0.155904029046793 rpy=1.57079632679489 -1.06806361303278 1.5707963267949 -> xyz=0.254228939952 0.136999999516020 -0.155904029536466 rpy=1.57079632679489 -1.06806361303278 1.5707963267949
- joint xj1_optical_joint: origin xyz=0 0 0 rpy=-1.5707963267949 0 -1.5707963267949 -> xyz=0 0 0 rpy=-1.570796326795 0 -1.570796326795
- joint xj2_optical_joint: origin xyz=0 0 0 rpy=-1.5707963267949 0 -1.5707963267949 -> xyz=0 0 0 rpy=-1.570796326795 0 -1.570796326795
- joint xj3_optical_joint: origin xyz=0 0 0 rpy=-1.5707963267949 0 -1.5707963267949 -> xyz=0 0 0 rpy=-1.570796326795 0 -1.570796326795
- joint xj4_optical_joint: origin xyz=0 0 0 rpy=-1.5707963267949 0 -1.5707963267949 -> xyz=0 0 0 rpy=-1.570796326795 0 -1.570796326795

Commit message: fix(sim): align pitch camera and vehicle forward

File: ros_ws/src/metro_description/urdf/subway_v2.urdf (robot description, URDF)
Before this commit: robot subway_v2, 27 links, 26 joints
Joints:
- joint base_footprint_to_base_link: origin xyz=0.010904028627 0.003428939952 0.214499211212 rpy=-1.570796326795 0 -1.570796326795 -> xyz=-0.010904028627 -0.003428939952 0.214499211212 rpy=-1.570796326795 0 1.570796326795
- joint w1_joint: axis 0 0 -1 -> 0 0 1
- joint w2_joint: axis 0 0 1 -> 0 0 -1
- joint w3_joint: axis 0 0 1 -> 0 0 -1
- joint w4_joint: axis 0 0 -1 -> 0 0 1

Commit message: fix(sim): align robot nose with forward motion

File: ros_ws/src/metro_description/urdf/subway_v2.urdf (robot description, URDF)
Before this commit: robot subway_v2, 27 links, 26 joints
Joints:
- joint base_footprint_to_base_link: origin xyz=-0.010904028627 -0.003428939952 0.214499211212 rpy=-1.570796326795 0 1.570796326795 -> xyz=0.010904028627 0.003428939952 0.214499211212 rpy=-1.570796326795 0 -1.570796326795
- joint w1_joint: axis 0 0 1 -> 0 0 -1
- joint w2_joint: axis 0 0 -1 -> 0 0 1
- joint w3_joint: axis 0 0 -1 -> 0 0 1
- joint w4_joint: axis 0 0 1 -> 0 0 -1

Commit message: feat(sim): 小车调转方向及接入 YOLO 测试 v1

File: ros_ws/src/metro_description/urdf/subway_v2.urdf (robot description, URDF)
Before this commit: robot subway_v2, 27 links, 26 joints
Joints:
- joint pitch_joint: origin xyz=0 0.01 0 rpy=3.14050535389669 -1.5707963267949 0 -> xyz=0 0.01 0 rpy=-1.83259571459394 1.5707963267949 0

Commit message: feat(platform): integrate multi-camera YOLO inspection workflow

File: ros_ws/src/metro_description/urdf/subway_v2.urdf (robot description, URDF)
Before this commit: robot subway_v2, 27 links, 26 joints
Joints:
- joint pitch_camera_sensor_joint: origin xyz=-0.077300002798 0.003299999982 0.087818765 rpy=1.5707963267949 -1.5707963267949 0 -> xyz=-0.077300002798 0.003299999982 0.087818765 rpy=-3.14159265358979 -0.260712087614 -1.57079632679489
- joint pitch_joint: origin xyz=0 0.01 0 rpy=-1.83259571459394 1.5707963267949 0 -> xyz=0 0.01 0 rpy=3.14050535389669 -1.5707963267949 0
- joint yaw_joint: origin xyz=-0.0738710600481814 -0.166 -0.0109040290468001 rpy=3.14159265358979 1.5707963267949 0 -> xyz=0.080728936235469 -0.166 0.033082880992946 rpy=3.14159265358979 -1.5707963267949 0

Commit message: fix(sim): aim side cameras at tunnel utilities

File: ros_ws/src/metro_description/urdf/subway_v2.urdf (robot description, URDF)
Before this commit: robot subway_v2, 27 links, 26 joints
Joints:
- joint xj1_camera_joint: origin xyz=0 0 0.018478 rpy=-1.5707963267949 -1.5707963267949 0 -> xyz=0 0 0.018478 rpy=-3.14159265358979 -1.13446401379631 1.5707963267949
- joint xj2_camera_joint: origin xyz=0 0 0.018478 rpy=-1.5707963267949 -1.5707963267949 0 -> xyz=0 0 0.018478 rpy=-3.14159265358979 -1.13446401379631 1.5707963267949

Commit message: fix(sim): stabilize articulated pitch and startup view

File: ros_ws/src/metro_description/urdf/subway_v2.urdf (robot description, URDF)
Before this commit: robot subway_v2, 27 links, 26 joints
Joints:
- joint pitch_camera_sensor_joint: origin xyz=-0.077300002798 0.003299999982 0.087818765 rpy=1.5707963267949 -1.5707963267949 0 -> xyz=-0.077300002798 0.003299999982 0.087818765 rpy=-3.14159265358979 -0.260712087614 -1.57079632679489
- joint pitch_joint: axis (none) -> -1 0 0; limit (none) -> lower=-0.261799387799149 upper=0.523598775598299 effort=10 velocity=0.5; origin xyz=0 0.01 0 rpy=-1.83259571459394 1.5707963267949 0 -> xyz=0 0.01 0 rpy=3.14050535389669 -1.5707963267949 0; type fixed -> revolute
- joint yaw_joint: origin xyz=-0.0738710600481814 -0.166 -0.0109040290468001 rpy=3.14159265358979 1.5707963267949 0 -> xyz=0.080728936235469 -0.166 0.033082880992946 rpy=3.14159265358979 -1.5707963267949 0

Commit message: feat(sim): package desktop app and harden inspection runtime

File: ros_ws/src/metro_description/urdf/subway_v2.urdf (robot description, URDF)
Before this commit: robot subway_v2, 27 links, 26 joints
Joints:
- joint pitch_camera_sensor_joint: origin xyz=-0.077300002798 0.003299999982 0.087818765 rpy=-3.14159265358979 -0.260712087614 -1.57079632679489 -> xyz=-0.077300002798 -0.025686200096 0.095551824230 rpy=-3.14159265358979 -0.260712087614 -1.57079632679489
- joint pitch_joint: limit lower=-0.261799387799149 upper=0.523598775598299 effort=10 velocity=0.5 -> lower=-0.261799387799149 upper=0.785398163397448 effort=10 velocity=0.5
- joint xj2_camera_joint: origin xyz=0 0 0.018478 rpy=-3.14159265358979 -1.13446401379631 1.5707963267949 -> xyz=0 0 0.082 rpy=-3.14159265358979 -1.13446401379631 1.5707963267949
- joint xj3_camera_joint: origin xyz=0 0 0.077 rpy=-1.5707963267949 -1.5707963267949 0 -> xyz=0 0 0.112 rpy=3.14159265358979 -1.30899693899575 1.5707963267949
