Commit message: feat(sim): preserve stable model annotation and desktop demo

File: ros_ws/src/metro_navigation_demo/urdf/gazebo_train_tf.urdf (robot description, URDF)
Before this commit: robot gazebo_train_tf, 11 links, 10 joints
Links:
- added link ground_camera_link; visual box size=0.08 0.06 0.05
- added link left_side_camera_link; visual box size=0.08 0.06 0.05
- added link right_side_camera_link; visual box size=0.08 0.06 0.05
- link camera_link: geometry visual box size=0.12 0.10 0.06; visual cylinder length=0.012 radius=0.018
Joints:
- added joint ground_camera_joint: type fixed, parent base_link, child ground_camera_link, origin xyz=1.10 0 1.05 rpy=0 1.05 0
- added joint left_side_camera_joint: type fixed, parent base_link, child left_side_camera_link, origin xyz=0.85 0.82 0.90 rpy=0 0.65 -0.20
- added joint right_side_camera_joint: type fixed, parent base_link, child right_side_camera_link, origin xyz=0.85 -0.82 0.90 rpy=0 0.65 0.20
- joint camera_joint: origin xyz=0.62 0 0.48 rpy=0 0 0 -> xyz=0.78 0 0.82 rpy=0 0.38 0
- joint camera_rgb_joint: origin xyz=0.10 0 0 rpy=0 0 0 -> xyz=0.06 0 0 rpy=0 0 0
